Commit message: add urdf

File: src/aero_description/urdf/rover_base.urdf.xacro (robot description, xacro)
@@ -30,5 +30,5 @@
       <geometry>
         <mesh
-          filename="package://aero_description/meshes/base_link.STL" />
+          filename="$(find aero_description)/meshes/base_link.STL" />
       </geometry>
       <material
@@ -44,5 +44,5 @@
       <geometry>
         <mesh
-          filename="package://aero_description/meshes/base_link.STL" />
+          filename="$(find aero_description)/meshes/base_link.STL" />
       </geometry>
     </collision>
@@ -75,19 +75,19 @@
       <geometry>
         <mesh
-          filename="package://aero_description/meshes/link_rf.STL" />
-      </geometry>
-      <material
-        name="">
-        <color
-          rgba="0.752941176470588 0.752941176470588 0.752941176470588 1" />
-      </material>
-    </visual>
-    <collision>
-      <origin
-        xyz="0 0 0"
-        rpy="0 0 0" />
-      <geometry>
-        <mesh
-          filename="package://aero_description/meshes/link_rf.STL" />
+          filename="$(find aero_description)/meshes/link_rf.STL" />
+      </geometry>
+      <material
+        name="">
+        <color
+          rgba="0.752941176470588 0.752941176470588 0.752941176470588 1" />
+      </material>
+    </visual>
+    <collision>
+      <origin
+        xyz="0 0 0"
+        rpy="0 0 0" />
+      <geometry>
+        <mesh
+          filename="$(find aero_description)/meshes/link_rf.STL" />
       </geometry>
     </collision>
@@ -128,19 +128,19 @@
       <geometry>
         <mesh
-          filename="package://aero_description/meshes/link_rb.STL" />
-      </geometry>
-      <material
-        name="">
-        <color
-          rgba="0.752941176470588 0.752941176470588 0.752941176470588 1" />
-      </material>
-    </visual>
-    <collision>
-      <origin
-        xyz="0 0 0"
-        rpy="0 0 0" />
-      <geometry>
-        <mesh
-          filename="package://aero_description/meshes/link_rb.STL" />
+          filename="$(find aero_description)/meshes/link_rb.STL" />
+      </geometry>
+      <material
+        name="">
+        <color
+          rgba="0.752941176470588 0.752941176470588 0.752941176470588 1" />
+      </material>
+    </visual>
+    <collision>
+      <origin
+        xyz="0 0 0"
+        rpy="0 0 0" />
+      <geometry>
+        <mesh
+          filename="$(find aero_description)/meshes/link_rb.STL" />
       </geometry>
     </collision>
@@ -181,19 +181,19 @@
       <geometry>
         <mesh
-          filename="package://aero_description/meshes/link_lf.STL" />
-      </geometry>
-      <material
-        name="">
-        <color
-          rgba="0.752941176470588 0.752941176470588 0.752941176470588 1" />
-      </material>
-    </visual>
-    <collision>
-      <origin
-        xyz="0 0 0"
-        rpy="0 0 0" />
-      <geometry>
-        <mesh
-          filename="package://aero_description/meshes/link_lf.STL" />
+          filename="$(find aero_description)/meshes/link_lf.STL" />
+      </geometry>
+      <material
+        name="">
+        <color
+          rgba="0.752941176470588 0.752941176470588 0.752941176470588 1" />
+      </material>
+    </visual>
+    <collision>
+      <origin
+        xyz="0 0 0"
+        rpy="0 0 0" />
+      <geometry>
+        <mesh
+          filename="$(find aero_description)/meshes/link_lf.STL" />
       </geometry>
     </collision>
@@ -234,19 +234,19 @@
       <geometry>
         <mesh
-          filename="package://aero_description/meshes/link_lb.STL" />
-      </geometry>
-      <material
-        name="">
-        <color
-          rgba="0.752941176470588 0.752941176470588 0.752941176470588 1" />
-      </material>
-    </visual>
-    <collision>
-      <origin
-        xyz="0 0 0"
-        rpy="0 0 0" />
-      <geometry>
-        <mesh
-          filename="package://aero_description/meshes/link_lb.STL" />
+          filename="$(find aero_description)/meshes/link_lb.STL" />
+      </geometry>
+      <material
+        name="">
+        <color
+          rgba="0.752941176470588 0.752941176470588 0.752941176470588 1" />
+      </material>
+    </visual>
+    <collision>
+      <origin
+        xyz="0 0 0"
+        rpy="0 0 0" />
+      <geometry>
+        <mesh
+          filename="$(find aero_description)/meshes/link_lb.STL" />
       </geometry>
     </collision>
